File: Hardware/MidiToCvConnectors/MidiToCvConnectors.kicad_pcb (KiCad board)
At the start: 2 copper layers, 81.3 x 109.2 mm, 18 parts, among them J1 AudioJack3, J10 AudioJack3, J11 AudioJack3, J12 AudioJack3, J2 AudioJack3, J2 DIN-5_180degree, J3 AudioJack3, J4 AudioJack3, J5 AudioJack3, J6 AudioJack3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

Commit message: software added
Parts:
- removed the J1 at (200.7, 48.3)
- removed the J1 at (174.0, 48.3)
- removed the J1 at (97.8, 61.6)
- removed the J1 at (188.0, 48.3)
- removed the J1 at (134.6, 41.8)
- removed U1: ATtiny84A-P, Package_DIP:DIP-14_W7.62mm
- J10: value AudioJack3 -> CV 4 OUT
- J11: value AudioJack3 -> GATE 4 OUT
- J12: value AudioJack3 -> Conn_01x02; footprint AudioJacks:Jack_3.5mm_QingPu_WQP-PJ301M-12_Vertical -> Connector_Wire:SolderWire-0.1sqmm_1x02_P3.6mm_D0.4mm_OD1mm
- J2, J3: value AudioJack3 -> Conn_01x08_Socket; footprint AudioJacks:Jack_3.5mm_QingPu_WQP-PJ301M-12_Vertical -> Connector_PinHeader_2.54mm:PinHeader_1x08_P2.54mm_Vertical; moved to B.Cu
- J4: value AudioJack3 -> CV 1 OUT
- J5: value AudioJack3 -> GATE 1 OUT
- J6: value AudioJack3 -> CV 2 OUT
- J7: value AudioJack3 -> GATE 2 OUT
- J8: value AudioJack3 -> CV 3 OUT
- J9: value AudioJack3 -> GATE 3 OUT
- moved J1 137.2 mm to (40.0, 63.5)
- moved J12 135.5 mm to (38.2, 52.1)
- moved J3 126.4 mm to (48.9, 152.4), turned to 90 degrees
- moved J10 119.4 mm to (33.0, 142.9)
- moved J4 119.4 mm to (33.0, 89.5)
- moved J6 119.4 mm to (33.0, 107.3)
- moved J8 119.4 mm to (33.0, 125.1)
- moved J2 117.5 mm to (31.1, 45.7), turned to -90 degrees
- moved J11 88.5 mm to (47.0, 142.9)
- moved J5 88.5 mm to (47.0, 89.5)
- moved J7 88.5 mm to (47.0, 107.3)
- moved J9 88.5 mm to (47.0, 125.1)
- renumbered J2 to J1
Connections:
- J10 pad S: (no net) -> GND
- J10 pad T: (no net) -> CV_4_OUT
- J10 pad TN: (no net) -> unconnected-(J10-PadTN)
- J11 pad S: (no net) -> GND
- J11 pad T: (no net) -> GATE_4_OUT
- J11 pad TN: (no net) -> unconnected-(J11-PadTN)
- J4 pad S: (no net) -> GND
- J4 pad T: (no net) -> CV_1_OUT
- J4 pad TN: (no net) -> unconnected-(J4-PadTN)
- J5 pad S: (no net) -> GND
- J5 pad T: (no net) -> GATE_1_OUT
- J5 pad TN: (no net) -> unconnected-(J5-PadTN)
- J6 pad S: (no net) -> GND
- J6 pad T: (no net) -> CV_2_OUT
- J6 pad TN: (no net) -> unconnected-(J6-PadTN)
- J7 pad S: (no net) -> GND
- J7 pad T: (no net) -> GATE_2_OUT
- J7 pad TN: (no net) -> unconnected-(J7-PadTN)
- J8 pad S: (no net) -> GND
- J8 pad T: (no net) -> CV_3_OUT
- J8 pad TN: (no net) -> unconnected-(J8-PadTN)
- J9 pad S: (no net) -> GND
- J9 pad T: (no net) -> GATE_3_OUT
- J9 pad TN: (no net) -> unconnected-(J9-PadTN)
Routing:
- net GATE_1_OUT: track 0.00 -> 70.2 mm
- net CV_1_OUT: track 0.00 -> 70.2 mm
- net GATE_2_OUT: track 0.00 -> 53.0 mm
- net CV_2_OUT: track 0.00 -> 52.9 mm
- net GATE_3_OUT: track 0.00 -> 35.7 mm
- net CV_3_OUT: track 0.00 -> 35.7 mm
- net MIDI_SINK: track 0.00 -> 20.8 mm
- net MIDI_SOURCE: track 0.00 -> 17.2 mm
- net GATE_4_OUT: track 0.00 -> 16.9 mm
- net CV_4_OUT: track 0.00 -> 16.9 mm
- added copper zone on B.Cu, net GND
- added copper zone on F.Cu, net GND
Other:
- board size 81.3 x 109.2 mm -> 29.2 x 109.2 mm
