File: Hardware/MidiToCvConnectors/MidiToCvConnectors.kicad_sch (KiCad schematic)
At the start: 3 parts, among them J1 AudioJack3, J2 DIN-5_180degree, U1 ATtiny84A-P

Commit message: software added
Parts:
- removed J1: AudioJack3, AudioJacks:Jack_3.5mm_QingPu_WQP-PJ301M-12_Vertical, symbol Connector:AudioJack3
- removed U1: ATtiny84A-P, Package_DIP:DIP-14_W7.62mm, symbol MCU_Microchip_ATtiny:ATtiny84A-P
- added J10: CV 4 OUT, AudioJacks:Jack_3.5mm_QingPu_WQP-PJ301M-12_Vertical, symbol Connector_Audio:AudioJack2_SwitchT
- added J11: GATE 4 OUT, AudioJacks:Jack_3.5mm_QingPu_WQP-PJ301M-12_Vertical, symbol Connector_Audio:AudioJack2_SwitchT
- added J12: Conn_01x02, Connector_Wire:SolderWire-0.1sqmm_1x02_P3.6mm_D0.4mm_OD1mm, symbol Connector_Generic:Conn_01x02
- added J2, J3: Conn_01x08_Socket, Connector_PinHeader_2.54mm:PinHeader_1x08_P2.54mm_Vertical, symbol Connector:Conn_01x08_Socket
- added J4: CV 1 OUT, AudioJacks:Jack_3.5mm_QingPu_WQP-PJ301M-12_Vertical, symbol Connector_Audio:AudioJack2_SwitchT
- added J5: GATE 1 OUT, AudioJacks:Jack_3.5mm_QingPu_WQP-PJ301M-12_Vertical, symbol Connector_Audio:AudioJack2_SwitchT
- added J6: CV 2 OUT, AudioJacks:Jack_3.5mm_QingPu_WQP-PJ301M-12_Vertical, symbol Connector_Audio:AudioJack2_SwitchT
- added J7: GATE 2 OUT, AudioJacks:Jack_3.5mm_QingPu_WQP-PJ301M-12_Vertical, symbol Connector_Audio:AudioJack2_SwitchT
- added J8: CV 3 OUT, AudioJacks:Jack_3.5mm_QingPu_WQP-PJ301M-12_Vertical, symbol Connector_Audio:AudioJack2_SwitchT
- added J9: GATE 3 OUT, AudioJacks:Jack_3.5mm_QingPu_WQP-PJ301M-12_Vertical, symbol Connector_Audio:AudioJack2_SwitchT
- renumbered J2 to J1
Connections:
- net GATE_1_OUT: now also J3.4 (Pin_4), J5.T
- net GND: now also J10.S, J11.S, J2.1 (Pin_1), J2.4 (Pin_4), J2.5 (Pin_5), J2.6 (Pin_6), J2.7 (Pin_7), J2.8 (Pin_8), J4.S, J5.S, J6.S, J7.S, J8.S, J9.S
- net MIDI_SINK: now also J12.2 (Pin_2), J2.2 (Pin_2)
- net MIDI_SOURCE: now also J12.1 (Pin_1), J2.3 (Pin_3)
- new net CV_1_OUT: J3.5 (Pin_5), J4.T
- new net CV_2_OUT: J3.6 (Pin_6), J6.T
- new net CV_3_OUT: J3.7 (Pin_7), J8.T
- new net CV_4_OUT: J10.T, J3.8 (Pin_8)
- new net GATE_2_OUT: J3.3 (Pin_3), J7.T
- new net GATE_3_OUT: J3.2 (Pin_2), J9.T
- new net GATE_4_OUT: J11.T, J3.1 (Pin_1)
