File: Hardware/MidiToCvFrontPanel/MidiToCvFrontPanel.kicad_pcb (KiCad board)
At the start: 2 copper layers, 37.9 x 128.5 mm, 16 parts, among them J1 AudioJack3, J10 AudioJack3, J11 AudioJack3, J12 AudioJack3, J13 Conn_02x05_Odd_Even, J14 Conn_01x06_Socket, J15 Conn_01x06_Socket, J2 AudioJack3, J3 AudioJack3, J4 AudioJack3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

Commit message: software added
Parts:
- removed H1: MountingHole, MountingHole:MountingHole_2.2mm_M2_ISO7380_Pad
- removed J1, J10, J11, J12, J2, J3, J4, J5, J6, J7, J8, J9: AudioJack3, AudioJacks:Jack_3.5mm_QingPu_WQP-PJ301M-12_Vertical
- removed J13: Conn_02x05_Odd_Even, Connector_IDC:IDC-Header_2x05_P2.54mm_Vertical
- removed J14, J15: Conn_01x06_Socket, Connector_PinSocket_2.54mm:PinSocket_1x06_P2.54mm_Vertical
Other:
- board size 37.9 x 128.5 mm -> 30 x 128.5 mm
- board text added: "CV 1"
- board text added: "CV 2"
- board text added: "CV 3"
- board text added: "CV 4"
- board text added: "GATE 1"
- board text added: "GATE 2"
- board text added: "GATE 3"
- board text added: "GATE 4"
- board text added: "JLCJLCJLCJLC"
- board text added: "MIDI IN"
- board text added: "MIDI TO CV"
