File: Hardware/MidiToCvLogic/MidiToCvLogic.kicad_pcb (KiCad board)
At the start: 2 copper layers, 56 parts, among them J1 Conn_02x05_Odd_Even, J2 Conn_01x06_Pin, J3 Conn_01x06_Socket, J4 Conn_01x06_Socket, J5 Conn_01x12_Socket, Q1 2N3904, Q2 2N3904, Q3 2N3904, Q4 2N3904, U1 LM7805_TO220, U2 ATmega328P-P, U3 6N138, U4 MCP4822, U5 MCP4822, U6 LM324, Y1 16MHz

Commit message: software added
Parts:
- removed H1, H2, H3, H4: MountingHole, MountingHole:MountingHole_2.2mm_M2_Pad
- removed J5: Conn_01x12_Socket, Connector_PinSocket_2.54mm:PinSocket_1x12_P2.54mm_Vertical
- added C7: 100nF, Capacitor_THT:C_Disc_D4.3mm_W1.9mm_P5.00mm, F.Cu at (50.2, 57.1)
- added R12: 3KΩ, Resistor_THT:R_Axial_DIN0207_L6.3mm_D2.5mm_P7.62mm_Horizontal, F.Cu at (47.6, 108.0)
- added R15: 3KΩ, Resistor_THT:R_Axial_DIN0207_L6.3mm_D2.5mm_P7.62mm_Horizontal, F.Cu at (47.6, 97.8)
- added R32: 10KΩ, Resistor_THT:R_Axial_DIN0207_L6.3mm_D2.5mm_P7.62mm_Horizontal, F.Cu at (54.6, 36.2)
- added R6: 3KΩ, Resistor_THT:R_Axial_DIN0207_L6.3mm_D2.5mm_P7.62mm_Horizontal, F.Cu at (47.6, 128.3)
- added R9: 3KΩ, Resistor_THT:R_Axial_DIN0207_L6.3mm_D2.5mm_P7.62mm_Horizontal, F.Cu at (47.6, 118.1)
- D2: footprint Diode_THT:D_DO-35_SOD27_P10.16mm_Horizontal -> Diode_THT:D_DO-35_SOD27_P7.62mm_Horizontal
- J1: moved to B.Cu
- J2: value Conn_01x06_Pin -> Conn_01x05; footprint Connector_PinHeader_2.54mm:PinHeader_1x06_P2.54mm_Horizontal -> Connector_JST:JST_PH_B5B-PH-K_1x05_P2.00mm_Vertical; moved to B.Cu
- J3, J4: value Conn_01x06_Socket -> Conn_01x08_Socket; footprint Connector_PinSocket_2.54mm:PinSocket_1x06_P2.54mm_Vertical -> Connector_PinSocket_2.54mm:PinSocket_1x08_P2.54mm_Vertical
- R10: renamed from R8; footprint Resistor_THT:R_Axial_DIN0207_L6.3mm_D2.5mm_P10.16mm_Horizontal -> Resistor_THT:R_Axial_DIN0207_L6.3mm_D2.5mm_P7.62mm_Horizontal
- R11: renamed from R9; value 10KΩ -> 4.7KΩ; footprint Resistor_THT:R_Axial_DIN0207_L6.3mm_D2.5mm_P10.16mm_Horizontal -> Resistor_THT:R_Axial_DIN0207_L6.3mm_D2.5mm_P7.62mm_Horizontal
- R13: renamed from R10; footprint Resistor_THT:R_Axial_DIN0207_L6.3mm_D2.5mm_P10.16mm_Horizontal -> Resistor_THT:R_Axial_DIN0207_L6.3mm_D2.5mm_P7.62mm_Horizontal
- R14: renamed from R11; value 10KΩ -> 4.7KΩ; footprint Resistor_THT:R_Axial_DIN0207_L6.3mm_D2.5mm_P10.16mm_Horizontal -> Resistor_THT:R_Axial_DIN0207_L6.3mm_D2.5mm_P7.62mm_Horizontal
- R16: renamed from R12; footprint Resistor_THT:R_Axial_DIN0207_L6.3mm_D2.5mm_P10.16mm_Horizontal -> Resistor_THT:R_Axial_DIN0207_L6.3mm_D2.5mm_P7.62mm_Horizontal
- R17: renamed from R13; footprint Resistor_THT:R_Axial_DIN0207_L6.3mm_D2.5mm_P10.16mm_Horizontal -> Resistor_THT:R_Axial_DIN0207_L6.3mm_D2.5mm_P7.62mm_Horizontal
- R18: renamed from R14; footprint Resistor_THT:R_Axial_DIN0207_L6.3mm_D2.5mm_P10.16mm_Horizontal -> Resistor_THT:R_Axial_DIN0207_L6.3mm_D2.5mm_P7.62mm_Horizontal
- R19: renamed from R15; footprint Resistor_THT:R_Axial_DIN0207_L6.3mm_D2.5mm_P10.16mm_Horizontal -> Resistor_THT:R_Axial_DIN0207_L6.3mm_D2.5mm_P7.62mm_Horizontal
- R20: renamed from R16; footprint Resistor_THT:R_Axial_DIN0207_L6.3mm_D2.5mm_P10.16mm_Horizontal -> Resistor_THT:R_Axial_DIN0207_L6.3mm_D2.5mm_P7.62mm_Horizontal
- R21: renamed from R17; footprint Resistor_THT:R_Axial_DIN0207_L6.3mm_D2.5mm_P10.16mm_Horizontal -> Resistor_THT:R_Axial_DIN0207_L6.3mm_D2.5mm_P7.62mm_Horizontal
- R22: renamed from R18; footprint Resistor_THT:R_Axial_DIN0207_L6.3mm_D2.5mm_P10.16mm_Horizontal -> Resistor_THT:R_Axial_DIN0207_L6.3mm_D2.5mm_P7.62mm_Horizontal
- R23: renamed from R19; footprint Resistor_THT:R_Axial_DIN0207_L6.3mm_D2.5mm_P10.16mm_Horizontal -> Resistor_THT:R_Axial_DIN0207_L6.3mm_D2.5mm_P7.62mm_Horizontal
- R24: renamed from R20; footprint Resistor_THT:R_Axial_DIN0207_L6.3mm_D2.5mm_P10.16mm_Horizontal -> Resistor_THT:R_Axial_DIN0207_L6.3mm_D2.5mm_P7.62mm_Horizontal
- R25: renamed from R21; footprint Resistor_THT:R_Axial_DIN0207_L6.3mm_D2.5mm_P10.16mm_Horizontal -> Resistor_THT:R_Axial_DIN0207_L6.3mm_D2.5mm_P7.62mm_Horizontal
- R26: renamed from R22; footprint Resistor_THT:R_Axial_DIN0207_L6.3mm_D2.5mm_P10.16mm_Horizontal -> Resistor_THT:R_Axial_DIN0207_L6.3mm_D2.5mm_P7.62mm_Horizontal
- R27: renamed from R23; footprint Resistor_THT:R_Axial_DIN0207_L6.3mm_D2.5mm_P10.16mm_Horizontal -> Resistor_THT:R_Axial_DIN0207_L6.3mm_D2.5mm_P7.62mm_Horizontal
- R28: renamed from R24; footprint Resistor_THT:R_Axial_DIN0207_L6.3mm_D2.5mm_P10.16mm_Horizontal -> Paul:R_Axial_DIN0207_L6.3mm_D2.5mm_P7.62mm_Horizontal_Thin
- R29: renamed from R25; footprint Resistor_THT:R_Axial_DIN0207_L6.3mm_D2.5mm_P10.16mm_Horizontal -> Paul:R_Axial_DIN0207_L6.3mm_D2.5mm_P7.62mm_Horizontal_Thin
- R30: renamed from R26; footprint Resistor_THT:R_Axial_DIN0207_L6.3mm_D2.5mm_P10.16mm_Horizontal -> Resistor_THT:R_Axial_DIN0207_L6.3mm_D2.5mm_P7.62mm_Horizontal
- R31: renamed from R27; footprint Resistor_THT:R_Axial_DIN0207_L6.3mm_D2.5mm_P10.16mm_Horizontal -> Resistor_THT:R_Axial_DIN0207_L6.3mm_D2.5mm_P7.62mm_Horizontal
- R4: footprint Resistor_THT:R_Axial_DIN0207_L6.3mm_D2.5mm_P10.16mm_Horizontal -> Resistor_THT:R_Axial_DIN0207_L6.3mm_D2.5mm_P7.62mm_Horizontal
- R5: value 10KΩ -> 4.7KΩ; footprint Resistor_THT:R_Axial_DIN0207_L6.3mm_D2.5mm_P10.16mm_Horizontal -> Resistor_THT:R_Axial_DIN0207_L6.3mm_D2.5mm_P7.62mm_Horizontal
- R7: renamed from R6; footprint Resistor_THT:R_Axial_DIN0207_L6.3mm_D2.5mm_P10.16mm_Horizontal -> Resistor_THT:R_Axial_DIN0207_L6.3mm_D2.5mm_P7.62mm_Horizontal
- R8: renamed from R7; value 10KΩ -> 4.7KΩ; footprint Resistor_THT:R_Axial_DIN0207_L6.3mm_D2.5mm_P10.16mm_Horizontal -> Resistor_THT:R_Axial_DIN0207_L6.3mm_D2.5mm_P7.62mm_Horizontal
- U1: footprint Package_TO_SOT_THT:TO-220-3_Horizontal_TabUp -> Package_TO_SOT_THT:TO-220-3_Vertical; moved to B.Cu
- U2: footprint Package_DIP:DIP-28_W7.62mm -> Package_DIP:DIP-28_W7.62mm_Socket
- Y1: footprint Crystal:Crystal_HC49-U_Vertical -> Crystal:Crystal_HC49-4H_Vertical
- moved R16 84.4 mm to (50.2, 135.9), turned to 90 degrees
- moved R5 79.5 mm to (45.1, 135.9), turned to 90 degrees
- moved R3 77.5 mm to (50.8, 46.4), turned to -90 degrees
- moved U1 76.8 mm to (50.2, 72.7)
- moved R4 76.1 mm to (42.5, 128.3), turned to -90 degrees
- moved R18 75.3 mm to (62.9, 135.9), turned to 90 degrees
- moved R1 74.3 mm to (50.8, 43.8), turned to 90 degrees
- moved R17 72.5 mm to (52.7, 128.3), turned to -90 degrees
- moved R2 72.1 mm to (54.6, 46.4), turned to -90 degrees
- moved R24 68.4 mm to (50.2, 115.6), turned to 90 degrees
- moved J3 67.9 mm to (43.8, 33.0), turned to 90 degrees
- moved U5 67.3 mm to (47.0, 56.5), turned to 180 degrees
- moved R19 63.7 mm to (60.3, 128.3), turned to -90 degrees
- moved J4 62.3 mm to (61.6, 139.7), turned to -90 degrees
- moved Q1 61.6 mm to (56.5, 133.3), turned to 90 degrees
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Connections:
- net -12V renamed -12V_IN
- net Net-(U4-VA) renamed /CV_1_PRE
- net Net-(U4-VB) renamed /CV_2_PRE
- net Net-(U5-VA) renamed /CV_3_PRE
- net Net-(U5-VB) renamed /CV_4_PRE
- C1 pad 1: Net-(D1-K) -> +12V
- C8 pad 1: +5V -> +12V
- D1 pad 1: Net-(D1-K) -> +12V
- D1 pad 2: +12V -> +12V_IN
- D2 pad 2: CV_1_OUT -> MIDI_SINK
- J1 pad 10: +12V -> +12V_IN
- J1 pad 9: +12V -> +12V_IN
- J3 pad 1: MIDI_SOURCE -> GND
- J3 pad 2: CV_1_OUT -> MIDI_SINK
- J3 pad 3: CV_1_OUT -> MIDI_SOURCE
- J3 pad 4: CV_1_OUT -> GND
- J3 pad 5: CV_3_OUT -> GND
- J3 pad 6: CV_4_OUT -> GND
- J4 pad 1: GND -> GATE_4_OUT
- J4 pad 2: unconnected-(J4-Pin_2-Pad2) -> GATE_3_OUT
- J4 pad 3: GATE_1_OUT -> GATE_2_OUT
- J4 pad 4: GATE_2_OUT -> GATE_1_OUT
- J4 pad 5: GATE_3_OUT -> CV_1_OUT
- J4 pad 6: GATE_4_OUT -> CV_2_OUT
- R11 pad 2: CV_3_OUT -> Net-(R11-Pad2)
- R14 pad 2: CV_4_OUT -> Net-(R14-Pad2)
- R3 pad 1: +5V -> RX
- R3 pad 2: RX -> +5V
- R5 pad 2: CV_1_OUT -> Net-(R5-Pad2)
- R8 pad 2: CV_1_OUT -> Net-(R8-Pad2)
- U1 pad 1: Net-(D1-K) -> +12V
- U3 pad 3: CV_1_OUT -> MIDI_SINK
- U6 pad 4: +5V -> +12V
- U6 pad 7: CV_1_OUT -> CV_2_OUT
Routing:
- net +5V: track 0.00 -> 161.8 mm
- net MOSI: track 0.00 -> 87.4 mm
- net SCK: track 0.00 -> 85.6 mm, vias 0 -> 1
- net GATE_1: track 0.00 -> 80.2 mm
- net CV_3_OUT: track 0.00 -> 76.3 mm
- net GATE_2: track 0.00 -> 66.2 mm
- net CV_2_OUT: track 0.00 -> 63.0 mm
- net Net-(U6C--): track 0.00 -> 59.5 mm
- net CV_4_OUT: track 0.00 -> 59.4 mm, vias 0 -> 1
- net RESET: track 0.00 -> 53.7 mm
- net GATE_3: track 0.00 -> 53.2 mm
- net Net-(U6A--): track 0.00 -> 52.6 mm
- net CV_1_OUT: track 0.00 -> 51.6 mm
- net /CV_3_PRE: track 0.00 -> 48.4 mm
- net GATE_4_OUT: track 0.00 -> 47.3 mm
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- added copper zone on B.Cu, net GND
- added copper zone on F.Cu, net GND
Other:
- board outline added: 29.2 x 109.2 mm
