File: Hardware/MidiToCvLogic/MidiToCvLogic.kicad_sch (KiCad schematic)
At the start: 57 parts, among them J1 Conn_02x05_Odd_Even, J2 Conn_01x06_Pin, J3 Conn_01x06_Socket, J4 Conn_01x06_Socket, J5 Conn_01x12_Socket, Q1 2N3904, Q2 2N3904, Q3 2N3904, Q4 2N3904, U1 LM7805_TO220, U2 ATmega328P-P, U3 6N138, U4 MCP4822, U5 MCP4822, U6 LM324, Y1 16MHz

Commit message: software added
Parts:
- removed H1, H2, H3, H4: MountingHole, MountingHole:MountingHole_2.2mm_M2_Pad, symbol Mechanical:MountingHole
- removed J2: Conn_01x06_Pin, Connector_PinHeader_2.54mm:PinHeader_1x06_P2.54mm_Horizontal, symbol Connector:Conn_01x06_Pin
- removed J3, J4: Conn_01x06_Socket, Connector_PinSocket_2.54mm:PinSocket_1x06_P2.54mm_Vertical, symbol Connector:Conn_01x06_Socket
- removed J5: Conn_01x12_Socket, Connector_PinSocket_2.54mm:PinSocket_1x12_P2.54mm_Vertical, symbol Connector:Conn_01x12_Socket
- added C7: 100nF, Capacitor_THT:C_Disc_D4.3mm_W1.9mm_P5.00mm, symbol Device:C
- added J2: Conn_01x05, Connector_JST:JST_PH_B5B-PH-K_1x05_P2.00mm_Vertical, symbol Connector_Generic:Conn_01x05
- added J3, J4: Conn_01x08_Socket, Connector_PinSocket_2.54mm:PinSocket_1x08_P2.54mm_Vertical, symbol Connector:Conn_01x08_Socket
- added R12, R15, R6, R9: 3KΩ, Resistor_THT:R_Axial_DIN0207_L6.3mm_D2.5mm_P7.62mm_Horizontal, symbol Device:R
- D2: footprint Diode_THT:D_DO-35_SOD27_P10.16mm_Horizontal -> Diode_THT:D_DO-35_SOD27_P7.62mm_Horizontal
- R10: renamed from R8; footprint Resistor_THT:R_Axial_DIN0207_L6.3mm_D2.5mm_P10.16mm_Horizontal -> Resistor_THT:R_Axial_DIN0207_L6.3mm_D2.5mm_P7.62mm_Horizontal
- R11: renamed from R9; value 10KΩ -> 4.7KΩ; footprint Resistor_THT:R_Axial_DIN0207_L6.3mm_D2.5mm_P10.16mm_Horizontal -> Resistor_THT:R_Axial_DIN0207_L6.3mm_D2.5mm_P7.62mm_Horizontal
- R13: renamed from R10; footprint Resistor_THT:R_Axial_DIN0207_L6.3mm_D2.5mm_P10.16mm_Horizontal -> Resistor_THT:R_Axial_DIN0207_L6.3mm_D2.5mm_P7.62mm_Horizontal
- R14: renamed from R11; value 10KΩ -> 4.7KΩ; footprint Resistor_THT:R_Axial_DIN0207_L6.3mm_D2.5mm_P10.16mm_Horizontal -> Resistor_THT:R_Axial_DIN0207_L6.3mm_D2.5mm_P7.62mm_Horizontal
- R16: renamed from R12; footprint Resistor_THT:R_Axial_DIN0207_L6.3mm_D2.5mm_P10.16mm_Horizontal -> Resistor_THT:R_Axial_DIN0207_L6.3mm_D2.5mm_P7.62mm_Horizontal
- R17: renamed from R13; footprint Resistor_THT:R_Axial_DIN0207_L6.3mm_D2.5mm_P10.16mm_Horizontal -> Resistor_THT:R_Axial_DIN0207_L6.3mm_D2.5mm_P7.62mm_Horizontal
- R18: renamed from R14; footprint Resistor_THT:R_Axial_DIN0207_L6.3mm_D2.5mm_P10.16mm_Horizontal -> Resistor_THT:R_Axial_DIN0207_L6.3mm_D2.5mm_P7.62mm_Horizontal
- R19: renamed from R15; footprint Resistor_THT:R_Axial_DIN0207_L6.3mm_D2.5mm_P10.16mm_Horizontal -> Resistor_THT:R_Axial_DIN0207_L6.3mm_D2.5mm_P7.62mm_Horizontal
- R20: renamed from R16; footprint Resistor_THT:R_Axial_DIN0207_L6.3mm_D2.5mm_P10.16mm_Horizontal -> Resistor_THT:R_Axial_DIN0207_L6.3mm_D2.5mm_P7.62mm_Horizontal
- R21: renamed from R17; footprint Resistor_THT:R_Axial_DIN0207_L6.3mm_D2.5mm_P10.16mm_Horizontal -> Resistor_THT:R_Axial_DIN0207_L6.3mm_D2.5mm_P7.62mm_Horizontal
- R22: renamed from R18; footprint Resistor_THT:R_Axial_DIN0207_L6.3mm_D2.5mm_P10.16mm_Horizontal -> Resistor_THT:R_Axial_DIN0207_L6.3mm_D2.5mm_P7.62mm_Horizontal
- R23: renamed from R19; footprint Resistor_THT:R_Axial_DIN0207_L6.3mm_D2.5mm_P10.16mm_Horizontal -> Resistor_THT:R_Axial_DIN0207_L6.3mm_D2.5mm_P7.62mm_Horizontal
- R24: renamed from R20; footprint Resistor_THT:R_Axial_DIN0207_L6.3mm_D2.5mm_P10.16mm_Horizontal -> Resistor_THT:R_Axial_DIN0207_L6.3mm_D2.5mm_P7.62mm_Horizontal
- R25: renamed from R21; footprint Resistor_THT:R_Axial_DIN0207_L6.3mm_D2.5mm_P10.16mm_Horizontal -> Resistor_THT:R_Axial_DIN0207_L6.3mm_D2.5mm_P7.62mm_Horizontal
- R26: renamed from R22; footprint Resistor_THT:R_Axial_DIN0207_L6.3mm_D2.5mm_P10.16mm_Horizontal -> Resistor_THT:R_Axial_DIN0207_L6.3mm_D2.5mm_P7.62mm_Horizontal
- R27: renamed from R23; footprint Resistor_THT:R_Axial_DIN0207_L6.3mm_D2.5mm_P10.16mm_Horizontal -> Resistor_THT:R_Axial_DIN0207_L6.3mm_D2.5mm_P7.62mm_Horizontal
- R28: renamed from R24; footprint Resistor_THT:R_Axial_DIN0207_L6.3mm_D2.5mm_P10.16mm_Horizontal -> Paul:R_Axial_DIN0207_L6.3mm_D2.5mm_P7.62mm_Horizontal_Thin
- R29: renamed from R25; footprint Resistor_THT:R_Axial_DIN0207_L6.3mm_D2.5mm_P10.16mm_Horizontal -> Paul:R_Axial_DIN0207_L6.3mm_D2.5mm_P7.62mm_Horizontal_Thin
- R30: renamed from R26; footprint Resistor_THT:R_Axial_DIN0207_L6.3mm_D2.5mm_P10.16mm_Horizontal -> Resistor_THT:R_Axial_DIN0207_L6.3mm_D2.5mm_P7.62mm_Horizontal
- R31: renamed from R27; footprint Resistor_THT:R_Axial_DIN0207_L6.3mm_D2.5mm_P10.16mm_Horizontal -> Resistor_THT:R_Axial_DIN0207_L6.3mm_D2.5mm_P7.62mm_Horizontal
- R32: renamed from R28; footprint Resistor_THT:R_Axial_DIN0207_L6.3mm_D2.5mm_P10.16mm_Horizontal -> Resistor_THT:R_Axial_DIN0207_L6.3mm_D2.5mm_P7.62mm_Horizontal
- R4: footprint Resistor_THT:R_Axial_DIN0207_L6.3mm_D2.5mm_P10.16mm_Horizontal -> Resistor_THT:R_Axial_DIN0207_L6.3mm_D2.5mm_P7.62mm_Horizontal
- R5: value 10KΩ -> 4.7KΩ; footprint Resistor_THT:R_Axial_DIN0207_L6.3mm_D2.5mm_P10.16mm_Horizontal -> Resistor_THT:R_Axial_DIN0207_L6.3mm_D2.5mm_P7.62mm_Horizontal
- R7: renamed from R6; footprint Resistor_THT:R_Axial_DIN0207_L6.3mm_D2.5mm_P10.16mm_Horizontal -> Resistor_THT:R_Axial_DIN0207_L6.3mm_D2.5mm_P7.62mm_Horizontal
- R8: renamed from R7; value 10KΩ -> 4.7KΩ; footprint Resistor_THT:R_Axial_DIN0207_L6.3mm_D2.5mm_P10.16mm_Horizontal -> Resistor_THT:R_Axial_DIN0207_L6.3mm_D2.5mm_P7.62mm_Horizontal
- U1: footprint Package_TO_SOT_THT:TO-220-3_Horizontal_TabUp -> Package_TO_SOT_THT:TO-220-3_Vertical
- U2: footprint Package_DIP:DIP-28_W7.62mm -> Package_DIP:DIP-28_W7.62mm_Socket
- Y1: footprint Crystal:Crystal_HC49-U_Vertical -> Crystal:Crystal_HC49-4H_Vertical
Connections:
- net +12V: now also C1.1, C8.1, D1.1 (K), U1.1 (VI), U6.4 (V+); no longer D1.2 (A), J1.10 (Pin_10), J1.9 (Pin_9)
- net +5V: now also R3.2, C7.2; no longer C8.1, R3.1, U6.4 (V+)
- net CV_1_OUT: now also J4.5 (Pin_5), R6.2; no longer D2.2 (A), R5.2, R8.2, U3.3 (C2), U6.7
- net CV_3_OUT: now also J4.7 (Pin_7), R12.2; no longer R11.2
- net CV_4_OUT: now also J4.8 (Pin_8), R15.2; no longer R14.2
- net GATE_1_OUT: now also J4.4 (Pin_4)
- net GATE_2_OUT: now also J4.3 (Pin_3)
- net GATE_3_OUT: now also J4.2 (Pin_2)
- net GATE_4_OUT: now also J4.1 (Pin_1)
- net GND: now also C7.1, J2.1 (Pin_1), J3.1 (Pin_1), J3.4 (Pin_4), J3.5 (Pin_5), J3.6 (Pin_6), J3.7 (Pin_7), J3.8 (Pin_8)
- net MIDI_SOURCE: now also J3.3 (Pin_3)
- net MISO: now also J2.3 (Pin_3)
- net MOSI: now also J2.4 (Pin_4)
- net RESET: now also J2.5 (Pin_5)
- net RX: now also R3.1; no longer R3.2
- net SCK: now also J2.2 (Pin_2)
- net CV_4_PRE: now reaches U5.6 (VB), U6.12 (+)
- net CV_3_PRE: now reaches U5.8 (VA), U6.10 (+)
- net CV_2_PRE: now reaches U4.6 (VB), U6.5 (+)
- net CV_1_PRE: now reaches U4.8 (VA), U6.3 (+)
- net -12V renamed -12V_IN
- new net: R14.2, R15.1
- new net: R11.2, R12.1
- new net: R5.2, R6.1
- new net: R8.2, R9.1
- new net +12V_IN: D1.2 (A), J1.10 (Pin_10), J1.9 (Pin_9)
- new net CV_2_OUT: J4.6 (Pin_6), R9.2, U6.7
- new net MIDI_SINK: D2.2 (A), J3.2 (Pin_2), U3.3 (C2)
- no-connect marks 1 -> 0
Other:
- moved on the sheet: R10, R11, R13, R14, R3, R4, R5, R7, R8, U6A, U6B, U6C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
